File: SS-XMAS-1.kicad_pcb (KiCad board)
At the start: 2 copper layers, 40.6 x 128.5 mm, 62 parts, among them J1 EURO_PWR_2x5, U1 ICM7555xP, U2 ICM7555xP

Commit message: Refactor
Parts:
- R1, R10, R11, R12, R13, R14, R15, R16, R18, R19, R2, R20, R21, R22, R27, R3, R4, R5, R6, R7, R8, R9: value 220K -> 330
- renumbered R17 to R330
Changed lines of the file:
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@@
 			)
 		)
-		(property "Value" "220K"
+		(property "Value" "330"
 			(at 5.08 0 0)
 			(layer "B.SilkS")
@@
 			)
 		)
-		(property "Value" "220K"
+		(property "Value" "330"
 			(at 5.08 0 0)
 			(layer "B.SilkS")
@@
 			)
 		)
-		(property "Value" "220K"
+		(property "Value" "330"
 			(at 5.08 0 0)
 			(layer "B.SilkS")
@@
 			)
 		)
-		(property "Value" "220K"
+		(property "Value" "330"
 			(at 5.08 0 0)
 			(layer "B.SilkS")
@@
 			)
 		)
-		(property "Value" "220K"
+		(property "Value" "330"
 			(at 5.08 0 0)
 			(layer "B.SilkS")
@@
 			)
 		)
-		(property "Value" "220K"
+		(property "Value" "330"
 			(at 5.08 0 0)
 			(layer "B.SilkS")
@@
 			)
 		)
-		(property "Value" "220K"
+		(property "Value" "330"
 			(at 5.08 0 0)
 			(layer "B.SilkS")
@@
 			)
 		)
-		(property "Value" "220K"
+		(property "Value" "330"
 			(at 5.08 0 0)
 			(layer "B.SilkS")
@@
 			)
 		)
-		(property "Value" "220K"
+		(property "Value" "330"
 			(at 5.08 0 0)
 			(layer "B.SilkS")
@@
 			)
 		)
-		(property "Value" "220K"
+		(property "Value" "330"
 			(at 5.08 0 0)
 			(layer "B.SilkS")
@@
 			)
 		)
-		(property "Value" "220K"
+		(property "Value" "330"
 			(at 5.08 0 0)
 			(layer "B.SilkS")
@@
 		(descr "Resistor, Axial_DIN0207 series, Axial, Horizontal, pin pitch=10.16mm, 0.25W = 1/4W, length*diameter=6.3*2.5mm^2, http://cdn-reichelt.de/documents/datenblatt/B400/1_4W%23YAG.pdf")
 		(tags "Resistor Axial_DIN0207 series Axial Horizontal pin pitch 10.16mm 0.25W = 1/4W length 6.3mm diameter 2.5mm")
-		(property "Reference" "R17"
+		(property "Reference" "R330"
 			(at 5.08 -2.54 0)
 			(layer "B.SilkS")
@@
 			)
 		)
-		(property "Value" "220K"
+		(property "Value" "330"
 			(at 5.08 0 75)
 			(layer "B.SilkS")
@@
 		(fp_line
 			(start 10.16 0.000001)
-			(end 8.23 0)
+			(end 8.230001 0)
 			(stroke
 				(width 0.1)
@@
 			)
 		)
-		(property "Value" "220K"
+		(property "Value" "330"
 			(at 5.08 0 0)
 			(layer "B.SilkS")
@@
 			)
 		)
-		(property "Value" "220K"
+		(property "Value" "330"
 			(at 5.08 0 0)
 			(layer "B.SilkS")
@@
 			)
 		)
-		(property "Value" "220K"
+		(property "Value" "330"
 			(at 5.08 0 0)
 			(layer "B.SilkS")
@@
 			)
 		)
-		(property "Value" "220K"
+		(property "Value" "330"
 			(at 5.08 0 -90)
 			(layer "B.SilkS")
@@
 			)
 		)
-		(property "Value" "220K"
+		(property "Value" "330"
 			(at 5.08 0 -90)
 			(layer "B.SilkS")
@@
 			)
 		)
-		(property "Value" "220K"
+		(property "Value" "330"
 			(at 5.08 0 0)
 			(layer "B.SilkS")
@@
 			)
 		)
-		(property "Value" "220K"
+		(property "Value" "330"
 			(at 5.08 0 0)
 			(layer "B.SilkS")
@@
 			)
 		)
-		(property "Value" "220K"
+		(property "Value" "330"
 			(at 5.08 0 -90)
 			(layer "B.SilkS")
@@
 			)
 		)
-		(property "Value" "220K"
+		(property "Value" "330"
 			(at 5.08 0 -90)
 			(layer "B.SilkS")
@@
 			)
 		)
-		(property "Value" "220K"
+		(property "Value" "330"
 			(at 5.08 0 0)
 			(layer "B.SilkS")
