File: SS-XMAS-1.kicad_sch (KiCad schematic)
At the start: 57 parts, among them J1 EURO_PWR_2x5, U1 ICM7555xP, U2 ICM7555xP

Commit message: Refactor
Parts:
- R1, R10, R11, R12, R13, R14, R15, R16, R17, R18, R19, R2, R20, R21, R22, R27, R3, R4, R5, R6, R7, R8, R9: value 220K -> 330
Changed lines of the file:
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@@
 			)
 		)
-		(property "Value" "220K"
+		(property "Value" "330"
 			(at 162.56 134.62 90)
 			(effects
@@
 			)
 		)
-		(property "Value" "220K"
+		(property "Value" "330"
 			(at 162.56 124.46 90)
 			(effects
@@
 			)
 		)
-		(property "Value" "220K"
+		(property "Value" "330"
 			(at 162.56 93.98 90)
 			(effects
@@
 			)
 		)
-		(property "Value" "220K"
+		(property "Value" "330"
 			(at 162.56 73.66 90)
 			(effects
@@
 			)
 		)
-		(property "Value" "220K"
+		(property "Value" "330"
 			(at 162.56 63.5 90)
 			(effects
@@
 			)
 		)
-		(property "Value" "220K"
+		(property "Value" "330"
 			(at 162.56 53.34 90)
 			(effects
@@
 			)
 		)
-		(property "Value" "220K"
+		(property "Value" "330"
 			(at 115.57 93.98 90)
 			(effects
@@
 			)
 		)
-		(property "Value" "220K"
+		(property "Value" "330"
 			(at 162.56 104.14 90)
 			(effects
@@
 			)
 		)
-		(property "Value" "220K"
+		(property "Value" "330"
 			(at 115.57 124.46 90)
 			(effects
@@
 			)
 		)
-		(property "Value" "220K"
+		(property "Value" "330"
 			(at 115.57 114.3 90)
 			(effects
@@
 			)
 		)
-		(property "Value" "220K"
+		(property "Value" "330"
 			(at 115.57 31.75 90)
 			(effects
@@
 			)
 		)
-		(property "Value" "220K"
+		(property "Value" "330"
 			(at 115.57 63.5 90)
 			(effects
@@
 			)
 		)
-		(property "Value" "220K"
+		(property "Value" "330"
 			(at 162.56 144.78 90)
 			(effects
@@
 			)
 		)
-		(property "Value" "220K"
+		(property "Value" "330"
 			(at 115.57 134.62 90)
 			(effects
@@
 			)
 		)
-		(property "Value" "220K"
+		(property "Value" "330"
 			(at 115.57 43.18 90)
 			(effects
@@
 			)
 		)
-		(property "Value" "220K"
+		(property "Value" "330"
 			(at 162.56 83.82 90)
 			(effects
@@
 			)
 		)
-		(property "Value" "220K"
+		(property "Value" "330"
 			(at 115.57 83.82 90)
 			(effects
@@
 			)
 		)
-		(property "Value" "220K"
+		(property "Value" "330"
 			(at 162.56 43.18 90)
 			(effects
@@
 			)
 		)
-		(property "Value" "220K"
+		(property "Value" "330"
 			(at 115.57 104.14 90)
 			(effects
@@
 			)
 		)
-		(property "Value" "220K"
+		(property "Value" "330"
 			(at 162.56 31.75 90)
 			(effects
@@
 			)
 		)
-		(property "Value" "220K"
+		(property "Value" "330"
 			(at 162.56 114.3 90)
 			(effects
@@
 			)
 		)
-		(property "Value" "220K"
+		(property "Value" "330"
 			(at 115.57 73.66 90)
 			(effects
@@
 			)
 		)
-		(property "Value" "220K"
+		(property "Value" "330"
 			(at 115.57 53.34 90)
 			(effects
